File: KiCadPCB/KiCadPCB.sch (KiCad schematic (older format))
At the start: 0 parts

Commit message: Started working on the schematic
Parts:
- added U?: ProMicro, symbol promicro:ProMicro
Changed lines of the file:
@@
 Comment4 ""
 $EndDescr
+$Comp
+L promicro:ProMicro U?
+U 1 1 615752A1
+P 1650 1800
+F 0 "U?" H 1650 2837 60  0000 C CNN
+F 1 "ProMicro" H 1650 2731 60  0000 C CNN
+F 2 "" H 1750 750 60  0000 C CNN
+F 3 "" H 1750 750 60  0000 C CNN
+	1    1650 1800
+	1    0    0    -1
+$EndComp
 $EndSCHEMATC
