File: KiCadPCB/KiCadPCB.sch (KiCad schematic (older format))
At the start: 1 part

Commit message: Added PCB files
Parts:
- added D1, D10, D11, D12, D13, D2, D3, D4, D5, D6, D7, D8, D9: 1N4148, Diode_THT:D_DO-35_SOD27_P7.62mm_Horizontal, symbol Device:D
- added D14: 1N4148, Diode_THT:D_DO-35_SOD27_P7.62mm_Horizontal, symbol Device:D_Small
- added SW1: M1, Button_Switch_Keyboard:SW_Cherry_MX_1.00u_PCB, symbol Switch:SW_Push
- added SW10: M10, Button_Switch_Keyboard:SW_Cherry_MX_1.00u_PCB, symbol Switch:SW_Push
- added SW11: M11, Button_Switch_Keyboard:SW_Cherry_MX_1.00u_PCB, symbol Switch:SW_Push
- added SW12: M12, Button_Switch_Keyboard:SW_Cherry_MX_1.00u_PCB, symbol Switch:SW_Push
- added SW13: M13, Button_Switch_Keyboard:SW_Cherry_MX_1.00u_PCB, symbol Switch:SW_Push
- added SW14: ENCODER, Rotary_Encoder:RotaryEncoder_Alps_EC12E-Switch_Vertical_H20mm, symbol Device:Rotary_Encoder_Switch
- added SW2: M2, Button_Switch_Keyboard:SW_Cherry_MX_1.00u_PCB, symbol Switch:SW_Push
- added SW3: M3, Button_Switch_Keyboard:SW_Cherry_MX_1.00u_PCB, symbol Switch:SW_Push
- added SW4: M4, Button_Switch_Keyboard:SW_Cherry_MX_1.00u_PCB, symbol Switch:SW_Push
- added SW5: M5, Button_Switch_Keyboard:SW_Cherry_MX_1.00u_PCB, symbol Switch:SW_Push
- added SW6: M6, Button_Switch_Keyboard:SW_Cherry_MX_1.00u_PCB, symbol Switch:SW_Push
- added SW7: M7, Button_Switch_Keyboard:SW_Cherry_MX_1.00u_PCB, symbol Switch:SW_Push
- added SW8: M8, Button_Switch_Keyboard:SW_Cherry_MX_1.00u_PCB, symbol Switch:SW_Push
- added SW9: M9, Button_Switch_Keyboard:SW_Cherry_MX_1.00u_PCB, symbol Switch:SW_Push
- U1: renamed from U?; footprint (none) -> promicro:ProMicro-NoSilk
Connections:
- net ROW0: now reaches U1.11 (B4)
- net ROW0: now also D1.2 (A), D2.2 (A), D3.2 (A), D4.2 (A), D5.2 (A), D6.2 (A), SW14.S1
- net ROW1: now reaches U1.12 (B5)
- net ROW1: now also D10.2 (A), D11.2 (A), D12.2 (A), D13.2 (A), D7.2 (A), D8.2 (A), D9.2 (A)
- net COL6: now reaches U1.13 (B6)
- net COL6: now also SW13.1, SW6.1
- net COL5: now reaches U1.14 (B2)
- net COL5: now also SW12.1, SW5.1
- net COL4: now reaches U1.15 (B3)
- net COL4: now also SW11.1, SW4.1
- net COL3: now reaches U1.16 (B1)
- net COL3: now also SW10.1, SW3.1
- net COL2: now reaches U1.17 (F7)
- net COL2: now also SW2.1, SW9.1
- net COL1: now reaches U1.18 (F6)
- net COL1: now also SW1.1, SW8.1
- net COL0: now reaches U1.19 (F5)
- net COL0: now also D14.1 (K), SW7.1
- net +5V: now reaches U1.21 (VCC)
- net GND: now reaches U1.23 (GND)
- net GND: now also U1.3 (GND), U1.4 (GND), SW14.C
- net at U1.7 (D4): now also SW14.B
- net at U1.8 (C6): now also SW14.A
- new net: D14.2 (A), SW14.S2
- new net: D5.1 (K), SW5.2
- new net: D4.1 (K), SW4.2
- new net: D6.1 (K), SW6.2
- new net: D3.1 (K), SW3.2
- new net: D2.1 (K), SW2.2
- new net: D1.1 (K), SW1.2
- new net: D12.1 (K), SW12.2
- new net: D11.1 (K), SW11.2
- new net: D13.1 (K), SW13.2
- new net: D10.1 (K), SW10.2
- new net: D9.1 (K), SW9.2
- new net: D8.1 (K), SW8.2
- new net: D7.1 (K), SW7.2
- no-connect marks 0 -> 9
Other:
- moved on the sheet: U1

Commit message: Added gerber files and updated the PCB files.
Parts:
- added H1, H2: MountingHole, MountingHole:MountingHole_3.2mm_M3, symbol Mechanical:MountingHole
Changed lines of the file:
@@
 Wire Wire Line
 	7750 1700 8600 1700
+$Comp
+L Mechanical:MountingHole H2
+U 1 1 618B365B
+P 10600 1150
+F 0 "H2" H 10700 1196 50  0000 L CNN
+F 1 "MountingHole" H 10700 1105 50  0000 L CNN
+F 2 "MountingHole:MountingHole_3.2mm_M3" H 10600 1150 50  0001 C CNN
+F 3 "~" H 10600 1150 50  0001 C CNN
+	1    10600 1150
+	1    0    0    -1
+$EndComp
+$Comp
+L Mechanical:MountingHole H1
+U 1 1 618B4503
+P 10600 900
+F 0 "H1" H 10700 946 50  0000 L CNN
+F 1 "MountingHole" H 10700 855 50  0000 L CNN
+F 2 "MountingHole:MountingHole_3.2mm_M3" H 10600 900 50  0001 C CNN
+F 3 "~" H 10600 900 50  0001 C CNN
+	1    10600 900
+	1    0    0    -1
+$EndComp
 $EndSCHEMATC

Commit message: updated firmware to a0, To Be Tested
Parts:
- U1: symbol promicro:ProMicro -> KiCadPCB-rescue:ProMicro-promicro
Changed lines of the file:
@@
 $EndDescr
 $Comp
-L promicro:ProMicro U1
+L KiCadPCB-rescue:ProMicro-promicro U1
 U 1 1 615752A1
 P 7050 2350
